File: KiCad/gloves dryer/gloves dryer.kicad_pcb (KiCad board)
At the start: 2 copper layers, 0 parts

Commit message: Finish V2 schematic with added button and first PCB layout, tolarance have to be double check before sending for manufacturing
Parts:
- added C1: 10u, Capacitor_THT:C_Radial_D5.0mm_H11.0mm_P2.00mm, F.Cu at (177.5, 66.0)
- added C2: 100u, Capacitor_THT:C_Radial_D6.3mm_H11.0mm_P2.50mm, F.Cu at (175.2, 74.0)
- added C3: 10p, Capacitor_THT:C_Disc_D3.0mm_W1.6mm_P2.50mm, F.Cu at (175.0, 79.5)
- added D1: 1N4007, Diode_THT:D_DO-41_SOD81_P10.16mm_Horizontal, F.Cu at (173.7, 69.0)
- added J1: Conn_01x03, Connector_PinHeader_2.00mm:PinHeader_1x03_P2.00mm_Vertical, F.Cu at (195.5, 67.0)
- added J4: PJ-114AH-SMT-TR, SAMESKY_PJ-114AH-SMT-TR:SAMESKY_PJ-114AH-SMT-TR, F.Cu at (169.0, 58.9)
- added J5: Conn_01x02, Connector_PinHeader_2.00mm:PinHeader_2x01_P2.00mm_Vertical, F.Cu at (186.5, 86.0)
- added J6: Conn_01x05, Connector_PinHeader_2.00mm:PinHeader_1x05_P2.00mm_Vertical, F.Cu at (192.5, 63.0)
- added J7: Conn_01x02, Connector_PinHeader_2.00mm:PinHeader_2x01_P2.00mm_Vertical, F.Cu at (193.0, 86.0)
- added Q1: PN2222A, Package_TO_SOT_THT:TO-92_Inline, F.Cu at (193.0, 81.5)
- added Q2: PN2222A, Package_TO_SOT_THT:TO-92_Inline, F.Cu at (193.0, 76.0)
- added R1: 1k, Resistor_THT:R_Axial_DIN0204_L3.6mm_D1.6mm_P7.62mm_Horizontal, F.Cu at (191.4, 59.8)
- added R2: 5k, Resistor_THT:R_Axial_DIN0204_L3.6mm_D1.6mm_P7.62mm_Horizontal, F.Cu at (194.5, 52.2)
- added R3: 1k, Resistor_THT:R_Axial_DIN0204_L3.6mm_D1.6mm_P7.62mm_Horizontal, F.Cu at (188.2, 59.8)
- added R4: 5k, Resistor_THT:R_Axial_DIN0204_L3.6mm_D1.6mm_P7.62mm_Horizontal, F.Cu at (185.0, 52.2)
- added R5: 220, Resistor_THT:R_Axial_DIN0204_L3.6mm_D1.6mm_P7.62mm_Horizontal, F.Cu at (181.8, 52.2)
- added R6: 10k, Resistor_THT:R_Axial_DIN0204_L3.6mm_D1.6mm_P7.62mm_Horizontal, F.Cu at (178.7, 52.2)
- added SW1: SW_Push_Dual, Button_Switch_THT:SW_PUSH_6mm_H5mm, F.Cu at (173.8, 84.0)
- added SW2: SW_Push_Dual, Button_Switch_THT:SW_PUSH_6mm_H5mm, F.Cu at (163.8, 84.0)
- added U1: PIC16F18126-I/P, PIC16F18126:PDIP14_P_MCH, F.Cu at (181.9, 64.5)
- added U2: AMS1117-5.0, Package_TO_SOT_SMD:SOT-223-3_TabPin2, F.Cu at (167.5, 76.0)
Routing:
- net /VDD_5V: track 0.00 -> 70.6 mm
- net /VDDG_12V: track 0.00 -> 45.0 mm
- net Net-(C3-Pad1): track 0.00 -> 34.9 mm
- net /MCLR: track 0.00 -> 26.7 mm
- net Net-(Q2-B): track 0.00 -> 25.3 mm
- net /BT1: track 0.00 -> 24.7 mm
- net /BT2: track 0.00 -> 23.3 mm
- net Net-(Q1-B): track 0.00 -> 23.2 mm
- net /IF1: track 0.00 -> 20.6 mm
- net /IF2: track 0.00 -> 20.3 mm
- net /F1-: track 0.00 -> 15.5 mm
- net /IO_SENS: track 0.00 -> 14.7 mm
- net /VDD_12V: track 0.00 -> 14.2 mm
- net /F2-: track 0.00 -> 7.33 mm
- net /DAT: track 0.00 -> 3.75 mm
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- added copper zone on B.Cu, net GND
- added copper zone on F.Cu, net GND
Other:
- board outline added: 36 x 40 mm
- board text added: "+"
- board text added: "-"
